File: cheapFeather.kicad_pcb (KiCad board)
At the start: 2 copper layers, 50.8 x 22.9 mm, 38 parts, among them J1 Conn_01x12, J2 Conn_01x16, J3 USB_B_Micro, J4 Conn_01x02, J5 Conn_01x02, Q1 BS170F, Q2 BS170F, Q3 BS170F, SW1 SW_Push, SW2 SW_Push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

Commit message: Changed cap. values
Parts:
- C5: value 1uF -> 4.7uF
Changed lines of the file:
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@@
     (add_net GND)
     (add_net "Net-(D2-Pad1)")
+    (add_net "Net-(J3-Pad4)")
     (add_net "Net-(R4-Pad1)")
     (add_net "Net-(R8-Pad1)")
+    (add_net "Net-(U1-Pad4)")
   )
   (module libs:USB_Micro_XKB (layer F.Cu)
@@
       (effects (font (size 1 1) (thickness 0.15)))
     )
-    (fp_text value 1uF (at 0 1.65) (layer F.Fab)
-      (effects (font (size 1 1) (thickness 0.15)))
-    )
+    (fp_text value 4.7uF (at 0 1.65) (layer F.Fab)
+      (effects (font (size 1 1) (thickness 0.15)))
+    )
